File: pyheld_pcb/power_section.kicad_sch (KiCad schematic)
At the start: 15 parts, among them J3 Conn_01x02, J3 USB_C_Receptacle_USB2.0

Commit message: Power section is almost finished
Parts:
- added C1: 100n, Capacitor_SMD:C_0603_1608Metric, symbol Device:C
- added D1: SS34, Diode_SMD:D_SMB, symbol Device:D_Schottky
- added D2: Green, Diode_SMD:D_0805_2012Metric, symbol Device:LED
- added D3: RED, Diode_SMD:D_0805_2012Metric, symbol Device:LED
- added L1: 22u, Inductor_SMD:L_0805_2012Metric, symbol Device:L
- added R2: 390k, Resistor_SMD:R_0603_1608Metric, symbol Device:R
- added R2: 51k, Resistor_SMD:R_0603_1608Metric, symbol Device:R
- added R3: 100, Resistor_SMD:R_0603_1608Metric, symbol Device:R
- added R4: 1k, Resistor_SMD:R_0603_1608Metric, symbol Device:R
- added R5, R6: 400, Resistor_SMD:R_0603_1608Metric, symbol Device:R
- added R7: 2k, Resistor_SMD:R_0603_1608Metric, symbol Device:R
- added SW7: SW_SPDT, work:SW_Slide_SPDT_wo_mount, symbol Switch:SW_SPDT
- added U3: DW01A, Package_TO_SOT_SMD:SOT-23-6, symbol newsymbols:DW01A
- added U3: AMS1117-3.3, Package_TO_SOT_SMD:SOT-223-3_TabPin2, symbol Regulator_Linear:AMS1117-3.3
- added U4: FS8502A, Package_SO:TSSOP-8_4.4x3mm_P0.65mm, symbol newsymbols:FS8502A
- added U5: TP4056, Package_SO:SOIC-8-1EP_3.9x4.9mm_P1.27mm_EP2.29x3mm_ThermalVias, symbol newsymbols:TP4056
- added U6: SDB628, Package_TO_SOT_SMD:SOT-23-6, symbol newsymbols:SDB628
Connections:
- net +3V3: now also U3.2 (VO)
- net +5V: now also D1.2 (A), R2.1, U3.3 (VI)
- net +BATT: now also R3.1, SW7.2 (B), U5.5 (BAT)
- net +VSW: now also L1.1, SW7.3 (C)
- net -BATT: now also U3.6 (GND), U4.2 (S1), U4.3 (S1)
- net GND: now also C1.1, R2.2, R4.2, R7.2, U3.1 (GND), U4.6 (S2), U4.7 (S2), U5.1 (TEMP), U5.3 (GND), U5.9 (GND)
- net VBUS: now also D2.2 (A), D3.2 (A), U5.4 (Vcc), U5.8 (CE)
- new net: R7.1, U5.2 (PROG)
- new net: R6.2, U5.6 (~{STDBY})
- new net: R5.2, U5.7 (~{CHRG})
- new net: C1.2, R3.2, U3.5 (VCC)
- new net: R2.1, R2.2
- new net: D1.1 (K), L1.2
- new net: U3.1 (OD), U4.4 (G1)
- new net: U3.3 (OC), U4.5 (G2)
- new net: D3.1 (K), R5.1
- new net: D2.1 (K), R6.1
- new net: R4.1, U3.2 (CS)
- no-connect marks 8 -> 12
Other:
- note added: "TODO USB C 5V mode"
