File: pyheld_pcb/pyheld_pcb.kicad_sch (KiCad schematic)
At the start: 0 parts

Commit message: Power section is almost finished
Other:
- sheet Power section ports: added +3V3, +5V, 5V enable, GND, U_BATT; removed none
Changed lines of the file:
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@@
+			)
+		)
+		(pin "+3V3" output
+			(at 49.53 45.72 180)
+			(effects
+				(font
+					(size 1.27 1.27)
+				)
+				(justify left)
+			)
+		)
+		(pin "+5V" output
+			(at 49.53 48.26 180)
+			(effects
+				(font
+					(size 1.27 1.27)
+				)
+				(justify left)
+			)
+		)
+		(pin "5V enable" input
+			(at 49.53 50.8 180)
+			(effects
+				(font
+					(size 1.27 1.27)
+				)
+				(justify left)
+			)
+		)
+		(pin "GND" output
+			(at 49.53 53.34 180)
+			(effects
+				(font
+					(size 1.27 1.27)
+				)
+				(justify left)
+			)
+		)
+		(pin "U_BATT" output
+			(at 49.53 55.88 180)
+			(effects
+				(font
+					(size 1.27 1.27)
+				)
+				(justify left)
 			)
 		)
